File: ledB_sch.brd (EAGLE design)
At the start: 22.9 x 22.9 mm, 7 parts

Commit message: gerber
Parts:
- renumbered LED1 to LED
Changed lines of the file:
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@@
 <?xml version="1.0" encoding="utf-8"?>
 <!DOCTYPE eagle SYSTEM "eagle.dtd">
-<eagle version="7.2.0">
+<eagle version="8.2.2">
 <drawing>
 <settings>
@@
 <setting verticaltext="up"/>
 </settings>
-<grid distance="10" unitdist="mil" unit="mil" style="lines" multiple="1" display="yes" altdistance="5" altunitdist="mil" altunit="mil"/>
+<grid distance="1" unitdist="mm" unit="mm" style="lines" multiple="1" display="yes" altdistance="5" altunitdist="mil" altunit="mil"/>
 <layers>
 <layer number="1" name="Top" color="4" fill="1" visible="yes" active="yes"/>
@@
 <plain>
 <circle x="11.43" y="11.43" radius="11.43" width="0.0254" layer="20"/>
+<wire x1="14" y1="20" x2="14" y2="18" width="0.1524" layer="21"/>
+<wire x1="15" y1="19" x2="13" y2="19" width="0.1524" layer="21"/>
+<wire x1="3.429" y1="18.415" x2="4.699" y2="18.415" width="0.1524" layer="21"/>
+<wire x1="4.064" y1="19.05" x2="4.064" y2="17.907" width="0.1524" layer="21"/>
+<wire x1="8.509" y1="20.193" x2="8.509" y2="18.923" width="0.1524" layer="21"/>
+<wire x1="2.413" y1="13.208" x2="3.683" y2="12.954" width="0.1524" layer="21"/>
+<wire x1="12.573" y1="1.651" x2="13.589" y2="1.651" width="0.1524" layer="21"/>
+<wire x1="13.081" y1="2.032" x2="13.081" y2="1.27" width="0.1524" layer="21"/>
+<wire x1="8.636" y1="1.524" x2="9.779" y2="1.524" width="0.1524" layer="21"/>
 </plain>
 <attributes>
@@
 <attribute name="VALUE" x="19.76948125" y="13.607146875" size="1.27" layer="27" ratio="10" rot="R115"/>
 </element>
-<element name="LED1" library="ledB_sch" package="LED5MM" value="" x="11.033" y="3.238" smashed="yes" rot="R180">
-<attribute name="NAME" x="13.573" y="5.4986" size="1.016" layer="25" ratio="10" rot="R180"/>
+<element name="LED" library="ledB_sch" package="LED5MM" value="" x="11.033" y="3.238" smashed="yes" rot="R180">
+<attribute name="NAME" x="12.573" y="5.4986" size="1.016" layer="25" ratio="10" rot="R180"/>
 <attribute name="VALUE" x="7.1976" y="6.3114" size="1.27" layer="27" ratio="10" rot="R180"/>
 </element>
 <element name="JP1" library="ledB_sch" package="1X02_OVAL" value="6V+" x="11.033" y="19.494" smashed="yes">
-<attribute name="VALUE" x="14.3388" y="18.145" size="1.016" layer="27" font="vector" ratio="10" rot="R90"/>
+<attribute name="VALUE" x="12.855" y="22.3388" size="1.016" layer="27" font="vector" ratio="10" rot="R180"/>
 </element>
 <element name="D1" library="ledB_sch" package="DO35-3" value="diode" x="17.383" y="7.048" smashed="yes" rot="R90">
@@
 <contactref element="JP1" pad="1"/>
 <contactref element="OPAMP" pad="4"/>
-<contactref element="LED1" pad="K"/>
+<contactref element="LED" pad="K"/>
 <contactref element="PIEZO" pad="1"/>
 <contactref element="R1" pad="1"/>
@@
 </signal>
 <signal name="N$5">
-<contactref element="LED1" pad="A"/>
+<contactref element="LED" pad="A"/>
 <contactref element="D1" pad="C"/>
 <wire x1="12.938" y1="3.238" x2="17.383" y2="3.238" width="0.4064" layer="1"/>
