File: ledB_sch.sch (EAGLE design)
At the start: 7 parts

Commit message: smd
Parts:
- D1: value diode -> 1N4001; device ledB_sch:1N4148-3 -> diode:DIODE-DO-214AC
- JP1: device ledB_sch:HEADER-1X2 -> ledB_sch:HEADER-1X2ROUND
- LED1: device ledB_sch:LED5MM -> ledB_sch:LED1206
- OPAMP: device ledB_sch:LM741P -> ledB_sch:LM741D
- R1, R2: device ledB_sch:R-US_0204/7 -> ledB_sch:R-US_M0805
Other:
- moved on the sheet: D1
Changed lines of the file:
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@@
 <?xml version="1.0" encoding="utf-8"?>
 <!DOCTYPE eagle SYSTEM "eagle.dtd">
-<eagle version="7.2.0">
+<eagle version="8.2.2">
 <drawing>
 <settings>
@@
 <layer number="97" name="Info" color="7" fill="1" visible="yes" active="yes"/>
 <layer number="98" name="Guide" color="6" fill="1" visible="yes" active="yes"/>
+<layer number="99" name="SpiceOrder" color="5" fill="1" visible="yes" active="yes"/>
 <layer number="100" name="Muster" color="7" fill="1" visible="no" active="no"/>
 <layer number="101" name="Patch_Top" color="12" fill="4" visible="no" active="yes"/>
@@
 </classes>
 <parts>
-<part name="OPAMP" library="ledB_sch" deviceset="*741" device="P" technology="LM" value="LM741"/>
-<part name="R1" library="ledB_sch" deviceset="R-US_" device="0204/7" value="10K"/>
-<part name="R2" library="ledB_sch" deviceset="R-US_" device="0204/7" value="10M"/>
-<part name="LED1" library="ledB_sch" deviceset="LED" device="5MM"/>
+<part name="OPAMP" library="ledB_sch" deviceset="*741" device="D" technology="LM" value="LM741"/>
+<part name="R1" library="ledB_sch" deviceset="R-US_" device="M0805" value="10K"/>
+<part name="R2" library="ledB_sch" deviceset="R-US_" device="M0805" value="10M"/>
+<part name="LED1" library="ledB_sch" deviceset="LED" device="1206"/>
 <part name="GND4" library="ledB_sch" deviceset="GND" device=""/>
-<part name="JP1" library="ledB_sch" deviceset="HEADER-1X2" device="" value="6V+"/>
+<part name="JP1" library="ledB_sch" deviceset="HEADER-1X2" device="ROUND" value="6V+"/>
 <part name="P+2" library="ledB_sch" deviceset="VCC" device=""/>
 <part name="GND2" library="ledB_sch" deviceset="GND" device=""/>
-<part name="D1" library="ledB_sch" deviceset="1N4148" device="-3" value="diode"/>
+<part name="D1" library="diode" library_urn="urn:adsk.eagle:library:210" deviceset="DIODE-" device="DO-214AC" value="1N4001"/>
 <part name="GND1" library="ledB_sch" deviceset="GND" device=""/>
 <part name="P+3" library="ledB_sch" deviceset="VCC" device=""/>
@@
 <instance part="P+2" gate="1" x="73.66" y="12.7" rot="R180"/>
 <instance part="GND2" gate="1" x="73.66" y="17.78" rot="R180"/>
-<instance part="D1" gate="G$1" x="63.5" y="27.94"/>
+<instance part="D1" gate="G$1" x="60.96" y="27.94"/>
 <instance part="GND1" gate="1" x="7.62" y="7.62" rot="MR0"/>
 <instance part="P+3" gate="1" x="38.1" y="38.1"/>
@@
 <pinref part="LED1" gate="G$1" pin="A"/>
 <pinref part="D1" gate="G$1" pin="C"/>
-<wire x1="66.04" y1="27.94" x2="71.12" y2="27.94" width="0.1524" layer="91"/>
+<wire x1="63.5" y1="27.94" x2="71.12" y2="27.94" width="0.1524" layer="91"/>
 </segment>
 </net>
@@
 which will not be processed correctly with this version.
 </note>
+<note version="8.2" severity="warning">
+Since Version 8.2, Eagle supports online libraries. The ids
+of those online libraries will not be understood (or retained)
+with this version.
+</note>
 </compatibility>
